Commit message: update

File: ros2_ws/src/workcell_description/urdf/workcell.urdf.xacro (robot description, xacro)
@@ -25,9 +25,9 @@
   <!-- Table 1 -->
   <xacro:moving_table prefix="t1_" parent="world">
-    <origin xyz="0 0.36 0" rpy="0 0 0"/>
+    <origin xyz="0 0.36 2.05" rpy="0 0 0"/>
   </xacro:moving_table>
   <!-- Table 2 -->
   <xacro:moving_table prefix="t2_" parent="world">
-    <origin xyz="0 -0.36 0" rpy="0 0 0"/>
+    <origin xyz="0 -0.36 2.05" rpy="0 0 0"/>
   </xacro:moving_table>
   <!-- ==================================== -->
@@ -36,5 +36,5 @@
   <ros2_control name="TableFakeHardware" type="system">
     <hardware>
-      <plugin>mock_components/MockSystem</plugin>
+      <plugin>mock_components/GenericSystem</plugin>
     </hardware>
     <joint name="t1_linear_joint">

Commit message: feat: Add sequence runner for ceilingArm demo choreography
- Implemented `run_sequence_demo.py` to drive the workcell through a fixed sequence involving table movements and arm/gripper actions.
- Introduced `moveit_controllers_per_arm.yaml` to define individual controllers for each arm and gripper, allowing for independent execution in RViz.
- Created `real_workcell.urdf.xacro` to support real hardware integration, forwarding necessary parameters for the Kinova driver.
- Launched `sequence_demo.launch.py` to start the sequence runner and dual table controller, with configurable parameters for gripper and table settings.
- Developed `single_rviz_workcell.launch.py` to enable switching between planning groups without relaunching, using real hardware configurations.
- Added `start_single_rviz.sh` script to streamline the launch process while avoiding broken environment overlays.
- Created `test_gripper_api.py` for direct testing of the Kinova gripper API, bypassing ROS to verify hardware functionality.

File: ros2_ws/src/workcell_description/urdf/workcell.urdf.xacro (robot description, xacro)
@@ -11,4 +11,11 @@
   <xacro:arg name="arm3_ip"           default="0.0.0.0"/>
   <xacro:arg name="arm4_ip"           default="0.0.0.0"/>
+  <!-- Per-arm mock override: default to the global flag, but each arm can be
+       mocked independently (e.g. mock an unreachable/powered-off arm so the
+       real ones still come up instead of the whole ros2_control_node aborting). -->
+  <xacro:arg name="arm1_fake"         default="$(arg use_fake_hardware)"/>
+  <xacro:arg name="arm2_fake"         default="$(arg use_fake_hardware)"/>
+  <xacro:arg name="arm3_fake"         default="$(arg use_fake_hardware)"/>
+  <xacro:arg name="arm4_fake"         default="$(arg use_fake_hardware)"/>
   <!-- ============================ -->
   <!-- Include table and Kinova URDF -->
@@ -67,22 +74,22 @@
   <!-- Arms Mounted on Table 1 -->
   <!-- ==================================== -->
-  <!-- Arm 1 (Left mount on Table 1) -->
-  <xacro:load_robot prefix="t1_a1_" parent="t1_mount_plate_left" arm="gen3_lite" dof="6" gripper="gen3_lite_2f" gripper_joint_name="right_finger_bottom_joint" use_fake_hardware="$(arg use_fake_hardware)" use_internal_bus_gripper_comm="true" gripper_max_velocity="100.0" gripper_max_force="100.0" vision="false" robot_ip="$(arg arm1_ip)" username="admin" password="admin" port="10000" port_realtime="10001" session_inactivity_timeout_ms="60000" connection_inactivity_timeout_ms="2000">
+  <!-- Arm 1 (t1_a1) — on table-1 RIGHT plate (left/right swapped to match real cell) -->
+  <xacro:load_robot prefix="t1_a1_" parent="t1_mount_plate_right" arm="gen3_lite" dof="6" gripper="gen3_lite_2f" gripper_joint_name="right_finger_bottom_joint" use_fake_hardware="$(arg arm1_fake)" use_internal_bus_gripper_comm="true" gripper_max_velocity="100.0" gripper_max_force="100.0" vision="false" robot_ip="$(arg arm1_ip)" username="admin" password="admin" port="10000" port_realtime="10001" session_inactivity_timeout_ms="60000" connection_inactivity_timeout_ms="2000">
+    <origin xyz="0 0 -0.025" rpy="3.14159 0 -1.5707963267948966"/>
+  </xacro:load_robot>
+  <!-- Arm 2 (t1_a2) — on table-1 LEFT plate (left/right swapped to match real cell) -->
+  <xacro:load_robot prefix="t1_a2_" parent="t1_mount_plate_left" arm="gen3_lite" dof="6" gripper="gen3_lite_2f" gripper_joint_name="right_finger_bottom_joint" use_fake_hardware="$(arg arm2_fake)" use_internal_bus_gripper_comm="true" gripper_max_velocity="100.0" gripper_max_force="100.0" vision="false" robot_ip="$(arg arm2_ip)" username="admin" password="admin" port="10000" port_realtime="10001" session_inactivity_timeout_ms="60000" connection_inactivity_timeout_ms="2000">
     <origin xyz="0 0 -0.025" rpy="3.14159 0 1.5707963267948966"/>
-  </xacro:load_robot>
-  <!-- Arm 2 (Right mount on Table 1) -->
-  <xacro:load_robot prefix="t1_a2_" parent="t1_mount_plate_right" arm="gen3_lite" dof="6" gripper="gen3_lite_2f" gripper_joint_name="right_finger_bottom_joint" use_fake_hardware="$(arg use_fake_hardware)" use_internal_bus_gripper_comm="true" gripper_max_velocity="100.0" gripper_max_force="100.0" vision="false" robot_ip="$(arg arm2_ip)" username="admin" password="admin" port="10000" port_realtime="10001" session_inactivity_timeout_ms="60000" connection_inactivity_timeout_ms="2000">
-    <origin xyz="0 0 -0.025" rpy="3.14159 0 -1.5707963267948966"/>
   </xacro:load_robot>
   <!-- ==================================== -->
   <!-- Arms Mounted on Table 2 -->
   <!-- ==================================== -->
-  <!-- Arm 3 (Left mount on Table 2) -->
-  <xacro:load_robot prefix="t2_a1_" parent="t2_mount_plate_left" arm="gen3_lite" dof="6" gripper="gen3_lite_2f" gripper_joint_name="right_finger_bottom_joint" use_fake_hardware="$(arg use_fake_hardware)" use_internal_bus_gripper_comm="true" gripper_max_velocity="100.0" gripper_max_force="100.0" vision="false" robot_ip="$(arg arm3_ip)" username="admin" password="admin" port="10000" port_realtime="10001" session_inactivity_timeout_ms="60000" connection_inactivity_timeout_ms="2000">
+  <!-- Arm 3 (t2_a1) — on table-2 RIGHT plate (left/right swapped to match real cell) -->
+  <xacro:load_robot prefix="t2_a1_" parent="t2_mount_plate_right" arm="gen3_lite" dof="6" gripper="gen3_lite_2f" gripper_joint_name="right_finger_bottom_joint" use_fake_hardware="$(arg arm3_fake)" use_internal_bus_gripper_comm="true" gripper_max_velocity="100.0" gripper_max_force="100.0" vision="false" robot_ip="$(arg arm3_ip)" username="admin" password="admin" port="10000" port_realtime="10001" session_inactivity_timeout_ms="60000" connection_inactivity_timeout_ms="2000">
+    <origin xyz="0 0 -0.025" rpy="3.14159 0 -1.5707963267948966"/>
+  </xacro:load_robot>
+  <!-- Arm 4 (t2_a2) — on table-2 LEFT plate (left/right swapped to match real cell) -->
+  <xacro:load_robot prefix="t2_a2_" parent="t2_mount_plate_left" arm="gen3_lite" dof="6" gripper="gen3_lite_2f" gripper_joint_name="right_finger_bottom_joint" use_fake_hardware="$(arg arm4_fake)" use_internal_bus_gripper_comm="true" gripper_max_velocity="100.0" gripper_max_force="100.0" vision="false" robot_ip="$(arg arm4_ip)" username="admin" password="admin" port="10000" port_realtime="10001" session_inactivity_timeout_ms="60000" connection_inactivity_timeout_ms="2000">
     <origin xyz="0 0 -0.025" rpy="3.14159 0 1.5707963267948966"/>
   </xacro:load_robot>
-  <!-- Arm 4 (Right mount on Table 2) -->
-  <xacro:load_robot prefix="t2_a2_" parent="t2_mount_plate_right" arm="gen3_lite" dof="6" gripper="gen3_lite_2f" gripper_joint_name="right_finger_bottom_joint" use_fake_hardware="$(arg use_fake_hardware)" use_internal_bus_gripper_comm="true" gripper_max_velocity="100.0" gripper_max_force="100.0" vision="false" robot_ip="$(arg arm4_ip)" username="admin" password="admin" port="10000" port_realtime="10001" session_inactivity_timeout_ms="60000" connection_inactivity_timeout_ms="2000">
-    <origin xyz="0 0 -0.025" rpy="3.14159 0 -1.5707963267948966"/>
-  </xacro:load_robot>
 </robot>

Commit message: refactor: Update workcell configuration and launch files for dual table controller integration

File: ros2_ws/src/workcell_description/urdf/workcell.urdf.xacro (robot description, xacro)
@@ -48,27 +48,12 @@
   </xacro:moving_table>
   <!-- ==================================== -->
-  <!-- Moving Tables Fake Hardware -->
+  <!-- Moving Tables Joint States -->
   <!-- ==================================== -->
-  <ros2_control name="TableFakeHardware" type="system">
-    <hardware>
-      <plugin>mock_components/GenericSystem</plugin>
-    </hardware>
-    <joint name="t1_linear_joint">
-      <command_interface name="position" />
-      <state_interface name="position" />
-    </joint>
-    <joint name="t1_rotation_joint">
-      <command_interface name="position" />
-      <state_interface name="position" />
-    </joint>
-    <joint name="t2_linear_joint">
-      <command_interface name="position" />
-      <state_interface name="position" />
-    </joint>
-    <joint name="t2_rotation_joint">
-      <command_interface name="position" />
-      <state_interface name="position" />
-    </joint>
-  </ros2_control>
+  <!-- The table joints are NOT under ros2_control. They are driven by the
+       dual_table_controller node (Modbus / fake) which publishes their
+       JointState on /table_joint_states; a joint_state_publisher aggregator
+       merges that into /joint_states for RViz. Keeping them out of
+       ros2_control makes dual_table_controller the single source of truth and
+       avoids a double-publisher conflict with joint_state_broadcaster. -->
   <!-- ==================================== -->
   <!-- Arms Mounted on Table 1 -->

File: ros2_ws/src/workcell_moveit_config/config/trailer_workcell.ros2_control.xacro (robot description, xacro)
@@ -204,32 +204,8 @@
                 <state_interface name="velocity"/>
             </joint>
-            <joint name="t1_linear_joint">
-                <command_interface name="position"/>
-                <state_interface name="position">
-                  <param name="initial_value">${initial_positions['t1_linear_joint']}</param>
-                </state_interface>
-                <state_interface name="velocity"/>
-            </joint>
-            <joint name="t1_rotation_joint">
-                <command_interface name="position"/>
-                <state_interface name="position">
-                  <param name="initial_value">${initial_positions['t1_rotation_joint']}</param>
-                </state_interface>
-                <state_interface name="velocity"/>
-            </joint>
-            <joint name="t2_linear_joint">
-                <command_interface name="position"/>
-                <state_interface name="position">
-                  <param name="initial_value">${initial_positions['t2_linear_joint']}</param>
-                </state_interface>
-                <state_interface name="velocity"/>
-            </joint>
-            <joint name="t2_rotation_joint">
-                <command_interface name="position"/>
-                <state_interface name="position">
-                  <param name="initial_value">${initial_positions['t2_rotation_joint']}</param>
-                </state_interface>
-                <state_interface name="velocity"/>
-            </joint>
+            <!-- Table joints (t1/t2 linear + rotation) are intentionally NOT
+                 declared here. They are driven by the dual_table_controller
+                 node and merged into /joint_states via a joint_state_publisher
+                 aggregator, so joint_state_broadcaster must not also own them. -->
         </ros2_control>
     </xacro:macro>

Commit message: Refactor take-bag and take-bottle demo scripts for absolute table motion
- Updated run_take_bag.py and run_take_bottle.py to use absolute table positions for movement, improving reliability across different starting positions.
- Introduced a new parameter `table_stable_samples` to ensure tables are settled before proceeding with the next steps.
- Modified the choreography in both demo scripts to reflect the new movement logic and added parallel table movement capabilities.
- Updated URDF to conditionally include fake hardware for tables based on the `use_fake_hardware` argument.
- Enhanced launch files for both take-bag and take-bottle demos to support spawning the dual_table_controller if not already running, preventing conflicts with serial port access.
- Added a Cartesian-velocity controller for arm_1 to facilitate compliant curtain pulling in the close curtain demo.

File: ros2_ws/src/workcell_description/urdf/workcell.urdf.xacro (robot description, xacro)
@@ -50,25 +50,32 @@
   <!-- Moving Tables Fake Hardware -->
   <!-- ==================================== -->
-  <ros2_control name="TableFakeHardware" type="system">
-    <hardware>
-      <plugin>mock_components/GenericSystem</plugin>
-    </hardware>
-    <joint name="t1_linear_joint">
-      <command_interface name="position" />
-      <state_interface name="position" />
-    </joint>
-    <joint name="t1_rotation_joint">
-      <command_interface name="position" />
-      <state_interface name="position" />
-    </joint>
-    <joint name="t2_linear_joint">
-      <command_interface name="position" />
-      <state_interface name="position" />
-    </joint>
-    <joint name="t2_rotation_joint">
-      <command_interface name="position" />
-      <state_interface name="position" />
-    </joint>
-  </ros2_control>
+  <!-- Only mock the table joints in fully-fake mode. On real hardware the table
+       joint states are owned and published by dual_table_controller (Modbus) on
+       /joint_states; a mock ros2_control system here would have joint_state_
+       broadcaster ALSO publish these joints as a constant 0, racing the real
+       values at ~5:1 and making the HUD / sequence _wait_for_table read 0. -->
+  <xacro:if value="$(arg use_fake_hardware)">
+    <ros2_control name="TableFakeHardware" type="system">
+      <hardware>
+        <plugin>mock_components/GenericSystem</plugin>
+      </hardware>
+      <joint name="t1_linear_joint">
+        <command_interface name="position" />
+        <state_interface name="position" />
+      </joint>
+      <joint name="t1_rotation_joint">
+        <command_interface name="position" />
+        <state_interface name="position" />
+      </joint>
+      <joint name="t2_linear_joint">
+        <command_interface name="position" />
+        <state_interface name="position" />
+      </joint>
+      <joint name="t2_rotation_joint">
+        <command_interface name="position" />
+        <state_interface name="position" />
+      </joint>
+    </ros2_control>
+  </xacro:if>
   <!-- ==================================== -->
   <!-- Arms Mounted on Table 1 -->
