Commit message: feat(isaac_sim): bridge workcell tables + polished scene in GUI bridge
- workcell.urdf.xacro: add sim_isaac TableTopicBased topic_based ros2_control for
  the 2 tables (t1/t2 linear+rotation) so they move in Isaac
- ros/ros2_controllers.yaml + bringup: add table_1/2_controller (JTC)
- ros2_bridge_gui.py: load polished environment (room + lights + work table)
  via polish.build_room/add_lights/recolor_tables

Verified: table_1 linear->0.15m, rotation->0.30rad in Isaac. Full workcell
(4 arms + 4 grippers + 2 tables) now ROS2-controllable in the simulation.

Co-Authored-By: Claude Opus 4.8 <noreply@anthropic.com>

File: ros2_ws/src/workcell_description/urdf/workcell.urdf.xacro (robot description, xacro)
@@ -81,4 +81,31 @@
     </ros2_control>
   </xacro:if>
+  <!-- Isaac Sim: drive the table joints through topic_based_ros2_control so they
+       move in the simulation (same /isaac_joint_* topics as the arms). -->
+  <xacro:if value="$(arg sim_isaac)">
+    <ros2_control name="TableTopicBased" type="system">
+      <hardware>
+        <plugin>topic_based_ros2_control/TopicBasedSystem</plugin>
+        <param name="joint_commands_topic">/isaac_joint_commands</param>
+        <param name="joint_states_topic">/isaac_joint_states</param>
+      </hardware>
+      <joint name="t1_linear_joint">
+        <command_interface name="position" />
+        <state_interface name="position" /><state_interface name="velocity" />
+      </joint>
+      <joint name="t1_rotation_joint">
+        <command_interface name="position" />
+        <state_interface name="position" /><state_interface name="velocity" />
+      </joint>
+      <joint name="t2_linear_joint">
+        <command_interface name="position" />
+        <state_interface name="position" /><state_interface name="velocity" />
+      </joint>
+      <joint name="t2_rotation_joint">
+        <command_interface name="position" />
+        <state_interface name="position" /><state_interface name="velocity" />
+      </joint>
+    </ros2_control>
+  </xacro:if>
   <!-- ==================================== -->
   <!-- Arms Mounted on Table 1 -->

Commit message: feat: real-hardware ros2_control bridge for tables, GNG self-filter fixes, new subsystem submodules
- dual_table_controller: optional topic_based_ros2_control bridge (table_hw_commands/states)
  so MoveIt can drive the real gantries via FollowJointTrajectory instead of only the
  move_dual_table service.
- gng_collision: re-filter the static background layer against live arm TF (history-based,
  larger radii) to stop permanent false self-collision from stale/incomplete captures.
- reach_fusion, target_cli, rgbd_perception launch: incidental fixes alongside the above.
- workcell URDF/moveit_config: controller + RViz config updates for the hardware bridge.
- add audio_common, whisper_ros, topic_based_ros2_control as tracked submodule gitlinks
  (matches existing ros2_kortex/livox_ros_driver2 convention) + yoloe-11m-seg.pt weights.

Co-Authored-By: Claude Sonnet 5 <noreply@anthropic.com>

File: ros2_ws/src/workcell_description/urdf/workcell.urdf.xacro (robot description, xacro)
@@ -21,4 +21,13 @@
   <xacro:arg name="arm3_fake"         default="$(arg use_fake_hardware)"/>
   <xacro:arg name="arm4_fake"         default="$(arg use_fake_hardware)"/>
+  <!-- Real-hardware gantry bridge (dual_table_controller to ros2_control via
+       topic_based_ros2_control). Requires the topic_based_ros2_control
+       package to actually be built in this workspace, NOT currently the
+       case (checked: `ros2 pkg prefix topic_based_ros2_control` fails), so
+       this defaults off. Flipping it on before that package exists makes
+       resource_manager fail to load the plugin and the WHOLE ros2_control_node
+       aborts (breaks real arm control too, not just the table): vendor and
+       colcon build topic_based_ros2_control first. -->
+  <xacro:arg name="enable_gantry_bridge" default="false"/>
   <!-- ============================ -->
   <!-- Include table and Kinova URDF -->
@@ -112,4 +121,39 @@
     </ros2_control>
   </xacro:if>
+  <!-- Real hardware, non-Isaac: drive the table joints through
+       topic_based_ros2_control against dual_table_controller's bridge
+       topics (table_hw_commands / table_hw_states), which translate goal
+       setpoints into real Modbus RTU go_to_absolute() calls. See
+       dual_table_controller.py's bridge.* params: bridge.enable must be
+       true (off by default) for this to actually drive the steppers. -->
+  <xacro:unless value="$(arg use_fake_hardware)">
+    <xacro:unless value="$(arg sim_isaac)">
+    <xacro:if value="$(arg enable_gantry_bridge)">
+      <ros2_control name="TableRealTopicBased" type="system">
+        <hardware>
+          <plugin>topic_based_ros2_control/TopicBasedSystem</plugin>
+          <param name="joint_commands_topic">table_hw_commands</param>
+          <param name="joint_states_topic">table_hw_states</param>
+        </hardware>
+        <joint name="t1_linear_joint">
+          <command_interface name="position" />
+          <state_interface name="position" />
+        </joint>
+        <joint name="t1_rotation_joint">
+          <command_interface name="position" />
+          <state_interface name="position" />
+        </joint>
+        <joint name="t2_linear_joint">
+          <command_interface name="position" />
+          <state_interface name="position" />
+        </joint>
+        <joint name="t2_rotation_joint">
+          <command_interface name="position" />
+          <state_interface name="position" />
+        </joint>
+      </ros2_control>
+    </xacro:if>
+    </xacro:unless>
+  </xacro:unless>
   <!-- ==================================== -->
   <!-- Arms Mounted on Table 1 -->
