Commit message: UPDATE

File: ros2_ws/src/workcell_description/urdf/moving_table.urdf.xacro (robot description, xacro)
@@ -37,5 +37,5 @@
       <origin xyz="0 0 0" rpy="0 0 0"/>
       <axis xyz="1 0 0"/>
-      <limit lower="-1.5" upper="1.5" effort="1000" velocity="0.5"/>
+      <limit lower="0.0" upper="1.5" effort="1000" velocity="0.5"/>
     </joint>
     <!-- Rotation bar -->

Commit message: Add Growing Neural Gas (GNG) implementation and evaluation tools
- Implemented GNG algorithm in `gng.py` for generating reachability maps.
- Added evaluation script `eval.py` for offline volume comparison and MoveIt IK benchmarking.
- Created `seed_ik.py` for generating joint configuration seeds using GNG.
- Developed `seed_server.py` to serve GNG joint configuration seeds via ROS topic.
- Introduced `train.py` for training the GNG model on FK datasets and annotating nodes with reachability stats.
- Added `visualize.py` to publish GNG maps as RViz markers.
- Created unit tests for GNG functionality in `test_gng.py`.
- Updated package configuration files for proper installation and resource management.
- Added resource directory for model files and configurations.

File: ros2_ws/src/workcell_description/urdf/moving_table.urdf.xacro (robot description, xacro)
@@ -37,5 +37,5 @@
       <origin xyz="0 0 0" rpy="0 0 0"/>
       <axis xyz="1 0 0"/>
-      <limit lower="0.0" upper="1.5" effort="1000" velocity="0.5"/>
+      <limit lower="0.0" upper="3.0" effort="1000" velocity="0.5"/>
     </joint>
     <!-- Rotation bar -->

File: ros2_ws/src/workcell_description/urdf/workcell_full.urdf (robot description, URDF)
Before this commit: robot trailer_workcell, 67 links, 66 joints
Links:
- link t1_a1_arm_link: geometry collision mesh filename=package://kortex_description/arms/gen3_lite/6dof/meshes/arm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; visual mesh filename=package://kortex_description/arms/gen3_lite/6dof/meshes/arm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
- link t1_a1_base_link: geometry collision mesh filename=package://kortex_description/arms/gen3_lite/6dof/meshes/bas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; visual mesh filename=package://kortex_description/arms/gen3_lite/6dof/meshes/bas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
- link t1_a1_forearm_link: geometry collision mesh filename=package://kortex_description/arms/gen3_lite/6dof/meshes/for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; visual mesh filename=package://kortex_description/arms/gen3_lite/6dof/meshes/for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
- link t1_a1_gripper_base_link: geometry collision mesh filename=package://kortex_description/grippers/gen3_lite_2f/meshes/g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; visual mesh filename=package://kortex_description/grippers/gen3_lite_2f/meshes/g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
- link t1_a1_left_finger_dist_link: geometry collision mesh filename=package://kortex_description/grippers/gen3_lite_2f/meshes/l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; visual mesh filename=package://kortex_description/grippers/gen3_lite_2f/meshes/l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
- link t1_a1_left_finger_prox_link: geometry collision mesh filename=package://kortex_description/grippers/gen3_lite_2f/meshes/l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; visual mesh filename=package://kortex_description/grippers/gen3_lite_2f/meshes/l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
- link t1_a1_lower_wrist_link: geometry collision mesh filename=package://kortex_description/arms/gen3_lite/6dof/meshes/low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; visual mesh filename=package://kortex_description/arms/gen3_lite/6dof/meshes/low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
- link t1_a1_right_finger_dist_link: geometry collision mesh filename=package://kortex_description/grippers/gen3_lite_2f/meshes/r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; visual mesh filename=package://kortex_description/grippers/gen3_lite_2f/meshes/r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
- link t1_a1_right_finger_prox_link: geometry collision mesh filename=package://kortex_description/grippers/gen3_lite_2f/meshes/r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; visual mesh filename=package://kortex_description/grippers/gen3_lite_2f/meshes/r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
- link t1_a1_shoulder_link: geometry collision mesh filename=package://kortex_description/arms/gen3_lite/6dof/meshes/sho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; visual mesh filename=package://kortex_description/arms/gen3_lite/6dof/meshes/sho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
- link t1_a1_upper_wrist_link: geometry collision mesh filename=package://kortex_description/arms/gen3_lite/6dof/meshes/upp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; visual mesh filename=package://kortex_description/arms/gen3_lite/6dof/meshes/upp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
- link t1_a2_arm_link: geometry collision mesh filename=package://kortex_description/arms/gen3_lite/6dof/meshes/arm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; visual mesh filename=package://kortex_description/arms/gen3_lite/6dof/meshes/arm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
- link t1_a2_base_link: geometry collision mesh filename=package://kortex_description/arms/gen3_lite/6dof/meshes/bas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; visual mesh filename=package://kortex_description/arms/gen3_lite/6dof/meshes/bas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
- link t1_a2_forearm_link: geometry collision mesh filename=package://kortex_description/arms/gen3_lite/6dof/meshes/for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; visual mesh filename=package://kortex_description/arms/gen3_lite/6dof/meshes/for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
- link t1_a2_gripper_base_link: geometry collision mesh filename=package://kortex_description/grippers/gen3_lite_2f/meshes/g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; visual mesh filename=package://kortex_description/grippers/gen3_lite_2f/meshes/g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
- link t1_a2_left_finger_dist_link: geometry collision mesh filename=package://kortex_description/grippers/gen3_lite_2f/meshes/l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; visual mesh filename=package://kortex_description/grippers/gen3_lite_2f/meshes/l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
- link t1_a2_left_finger_prox_link: geometry collision mesh filename=package://kortex_description/grippers/gen3_lite_2f/meshes/l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; visual mesh filename=package://kortex_description/grippers/gen3_lite_2f/meshes/l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
- link t1_a2_lower_wrist_link: geometry collision mesh filename=package://kortex_description/arms/gen3_lite/6dof/meshes/low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; visual mesh filename=package://kortex_description/arms/gen3_lite/6dof/meshes/low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
- link t1_a2_right_finger_dist_link: geometry collision mesh filename=package://kortex_description/grippers/gen3_lite_2f/meshes/r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; visual mesh filename=package://kortex_description/grippers/gen3_lite_2f/meshes/r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
- link t1_a2_right_finger_prox_link: geometry collision mesh filename=package://kortex_description/grippers/gen3_lite_2f/meshes/r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; visual mesh filename=package://kortex_description/grippers/gen3_lite_2f/meshes/r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
- link t1_a2_shoulder_link: geometry collision mesh filename=package://kortex_description/arms/gen3_lite/6dof/meshes/sho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; visual mesh filename=package://kortex_description/arms/gen3_lite/6dof/meshes/sho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
- link t1_a2_upper_wrist_link: geometry collision mesh filename=package://kortex_description/arms/gen3_lite/6dof/meshes/upp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; visual mesh filename=package://kortex_description/arms/gen3_lite/6dof/meshes/upp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
- link t2_a1_arm_link: geometry collision mesh filename=package://kortex_description/arms/gen3_lite/6dof/meshes/arm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; visual mesh filename=package://kortex_description/arms/gen3_lite/6dof/meshes/arm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
- link t2_a1_base_link: geometry collision mesh filename=package://kortex_description/arms/gen3_lite/6dof/meshes/bas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; visual mesh filename=package://kortex_description/arms/gen3_lite/6dof/meshes/bas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
- link t2_a1_forearm_link: geometry collision mesh filename=package://kortex_description/arms/gen3_lite/6dof/meshes/for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; visual mesh filename=package://kortex_description/arms/gen3_lite/6dof/meshes/for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
- link t2_a1_gripper_base_link: geometry collision mesh filename=package://kortex_description/grippers/gen3_lite_2f/meshes/g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; visual mesh filename=package://kortex_description/grippers/gen3_lite_2f/meshes/g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
- link t2_a1_left_finger_dist_link: geometry collision mesh filename=package://kortex_description/grippers/gen3_lite_2f/meshes/l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; visual mesh filename=package://kortex_description/grippers/gen3_lite_2f/meshes/l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
- link t2_a1_left_finger_prox_link: geometry collision mesh filename=package://kortex_description/grippers/gen3_lite_2f/meshes/l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; visual mesh filename=package://kortex_description/grippers/gen3_lite_2f/meshes/l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
- link t2_a1_lower_wrist_link: geometry collision mesh filename=package://kortex_description/arms/gen3_lite/6dof/meshes/low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; visual mesh filename=package://kortex_description/arms/gen3_lite/6dof/meshes/low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
- link t2_a1_right_finger_dist_link: geometry collision mesh filename=package://kortex_description/grippers/gen3_lite_2f/meshes/r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; visual mesh filename=package://kortex_description/grippers/gen3_lite_2f/meshes/r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
- link t2_a1_right_finger_prox_link: geometry collision mesh filename=package://kortex_description/grippers/gen3_lite_2f/meshes/r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; visual mesh filename=package://kortex_description/grippers/gen3_lite_2f/meshes/r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
- link t2_a1_shoulder_link: geometry collision mesh filename=package://kortex_description/arms/gen3_lite/6dof/meshes/sho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; visual mesh filename=package://kortex_description/arms/gen3_lite/6dof/meshes/sho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
- link t2_a1_upper_wrist_link: geometry collision mesh filename=package://kortex_description/arms/gen3_lite/6dof/meshes/upp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; visual mesh filename=package://kortex_description/arms/gen3_lite/6dof/meshes/upp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
- link t2_a2_arm_link: geometry collision mesh filename=package://kortex_description/arms/gen3_lite/6dof/meshes/arm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; visual mesh filename=package://kortex_description/arms/gen3_lite/6dof/meshes/arm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
- link t2_a2_base_link: geometry collision mesh filename=package://kortex_description/arms/gen3_lite/6dof/meshes/bas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; visual mesh filename=package://kortex_description/arms/gen3_lite/6dof/meshes/bas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
- link t2_a2_forearm_link: geometry collision mesh filename=package://kortex_description/arms/gen3_lite/6dof/meshes/for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; visual mesh filename=package://kortex_description/arms/gen3_lite/6dof/meshes/for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
- link t2_a2_gripper_base_link: geometry collision mesh filename=package://kortex_description/grippers/gen3_lite_2f/meshes/g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; visual mesh filename=package://kortex_description/grippers/gen3_lite_2f/meshes/g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
- link t2_a2_left_finger_dist_link: geometry collision mesh filename=package://kortex_description/grippers/gen3_lite_2f/meshes/l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; visual mesh filename=package://kortex_description/grippers/gen3_lite_2f/meshes/l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
- link t2_a2_left_finger_prox_link: geometry collision mesh filename=package://kortex_description/grippers/gen3_lite_2f/meshes/l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; visual mesh filename=package://kortex_description/grippers/gen3_lite_2f/meshes/l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
- link t2_a2_lower_wrist_link: geometry collision mesh filename=package://kortex_description/arms/gen3_lite/6dof/meshes/low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; visual mesh filename=package://kortex_description/arms/gen3_lite/6dof/meshes/low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
- link t2_a2_right_finger_dist_link: geometry collision mesh filename=package://kortex_description/grippers/gen3_lite_2f/meshes/r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; visual mesh filename=package://kortex_description/grippers/gen3_lite_2f/meshes/r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
- link t2_a2_right_finger_prox_link: geometry collision mesh filename=package://kortex_description/grippers/gen3_lite_2f/meshes/r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; visual mesh filename=package://kortex_description/grippers/gen3_lite_2f/meshes/r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
- link t2_a2_shoulder_link: geometry collision mesh filename=package://kortex_description/arms/gen3_lite/6dof/meshes/sho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; visual mesh filename=package://kortex_description/arms/gen3_lite/6dof/meshes/sho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
- link t2_a2_upper_wrist_link: geometry collision mesh filename=package://kortex_description/arms/gen3_lite/6dof/meshes/upp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; visual mesh filename=package://kortex_description/arms/gen3_lite/6dof/meshes/upp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
Joints:
- joint t1_linear_joint: limit lower=-1.5 upper=1.5 effort=1000 velocity=0.5 -> lower=0.0 upper=3.0 effort=1000 velocity=0.5

Commit message: Add reachability analysis and visualization nodes
- Implemented `reachability_check.py` to classify detected objects as reachable or not based on GNG reachability maps.
- Introduced `reachability_cloud.py` for per-object reachability analysis, supporting both voxel and point cloud modes.
- Created `seg_cloud.py` to publish a colorized 3D point cloud based on instance segmentation.
- Added `seg_colorizer.py` to convert instance segmentation labels to RGB colors for visualization.
- Developed `table_collision.py` to publish a static collision box representing the mapped work table for MoveIt integration.

File: ros2_ws/src/workcell_description/urdf/moving_table.urdf.xacro (robot description, xacro)
@@ -37,5 +37,5 @@
       <origin xyz="0 0 0" rpy="0 0 0"/>
       <axis xyz="1 0 0"/>
-      <limit lower="0.0" upper="3.0" effort="1000" velocity="0.5"/>
+      <limit lower="0.0" upper="2.0" effort="1000" velocity="0.5"/>
     </joint>
     <!-- Rotation bar -->

File: ros2_ws/src/workcell_description/urdf/workcell_full.urdf (robot description, URDF)
Before this commit: robot trailer_workcell, 67 links, 66 joints
Joints:
- joint t1_linear_joint: limit lower=0.0 upper=3.0 effort=1000 velocity=0.5 -> lower=0.0 upper=2.0 effort=1000 velocity=0.5
- joint t2_linear_joint: limit lower=-1.5 upper=1.5 effort=1000 velocity=0.5 -> lower=0.0 upper=2.0 effort=1000 velocity=0.5
