Commit message: urdf(jalanB): add rail friction/damping model to gantry joints
Jalan B step 1: give the rigid-body energy model a friction path so J can be
recalibrated to a realistic energy (frictionless model has R^2=0.055 vs traj_energy).
Coulomb friction = mu*N (mu=0.15; carried mass 18.77 kg linear / 13.77 kg rotation);
linear friction=27.6 N damping=1.4, rotation friction=2.03 Nm damping=0.10. These are
MODEL ASSUMPTIONS (sensitivity mu in {0.10,0.15,0.20}), not measured hardware -- report
as such, never as real motor energy. Regenerated workcell_full.urdf to match.

Co-Authored-By: Claude Opus 4.8 <noreply@anthropic.com>

File: ros2_ws/src/workcell_description/urdf/moving_table.urdf.xacro (robot description, xacro)
@@ -32,4 +32,14 @@
     </link>
     <!-- Linear slide -->
+    <!-- MODEL ASSUMPTION (not measured hardware data, added 2026-07-16 "Jalan B" to
+         give the rigid-body energy model a friction path; report as a sensitivity
+         in the paper, never as real motor energy):
+         Coulomb friction = mu * N, N = carried weight * g. Carried mass = platform
+         (5.0) + rotation_link (3.0) + 2x mount_plate (0.2 each) + 2x Kinova Gen3
+         Lite arm+gripper (~5.19 kg each, from kortex_description link masses)
+         = 18.77 kg -> N = 184.2 N. mu = 0.15 (mid of typical linear-guide range
+         0.10-0.20) -> friction = 27.6 N. Viscous damping set to 5% of the Coulomb
+         term (1.4 N*s/m) as a small secondary term. Sensitivity: mu in {0.10,
+         0.15, 0.20} -> friction in {18.4, 27.6, 36.8} N. -->
     <joint name="${prefix}linear_joint" type="prismatic">
       <parent link="${prefix}base_link"/>
@@ -37,4 +47,5 @@
       <origin xyz="0 0 0" rpy="0 0 0"/>
       <axis xyz="1 0 0"/>
+      <dynamics damping="1.4" friction="27.6"/>
       <limit lower="0.0" upper="2.0" effort="1000" velocity="0.5"/>
     </joint>
@@ -63,4 +74,11 @@
     </joint> -->
     <!-- Rotating joint (instead of fixed) -->
+    <!-- MODEL ASSUMPTION (not measured; same 2026-07-16 "Jalan B" note as above):
+         Coulomb friction torque = mu * N * r_bearing. Carried mass excludes the
+         platform (rotation_link + 2x mount_plate + 2x arm+gripper) = 13.77 kg
+         -> N = 135.1 N. mu = 0.15 (same family as the linear guide). r_bearing =
+         0.10 m, an assumed effective slew-bearing radius (not from any drawing)
+         -> friction = 2.03 Nm. Viscous damping = 5% of that (0.10 Nm*s/rad).
+         Sensitivity: mu in {0.10, 0.15, 0.20} -> friction in {1.35, 2.03, 2.70} Nm. -->
     <joint name="${prefix}rotation_joint" type="revolute">
       <parent link="${prefix}platform_link"/>
@@ -68,4 +86,5 @@
       <origin xyz="0 0 -${0.065/2 + 0.015/2}" rpy="0 0 ${pi/2}"/> <!-- default 90° -->
       <axis xyz="0 0 1"/> <!-- rotate around Z -->
+      <dynamics damping="0.10" friction="2.03"/>
       <limit lower="${-pi}" upper="${pi}" effort="10" velocity="1.0"/> <!-- ±180° travel -->
     </joint>

File: ros2_ws/src/workcell_description/urdf/workcell_full.urdf (robot description, URDF)
Before this commit: robot trailer_workcell, 67 links, 66 joints
Links:
- link t1_a1_gripper_base_link: geometry collision mesh filename=file:///srv/data/users/raditya/arm_WS/ceiling_arm/ros2_ws/i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; visual mesh filename=file:///srv/data/users/raditya/arm_WS/ceiling_arm/ros2_ws/i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
- link t1_a1_left_finger_dist_link: geometry collision mesh filename=file:///srv/data/users/raditya/arm_WS/ceiling_arm/ros2_ws/i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; visual mesh filename=file:///srv/data/users/raditya/arm_WS/ceiling_arm/ros2_ws/i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
- link t1_a1_left_finger_prox_link: geometry collision mesh filename=file:///srv/data/users/raditya/arm_WS/ceiling_arm/ros2_ws/i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; visual mesh filename=file:///srv/data/users/raditya/arm_WS/ceiling_arm/ros2_ws/i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
- link t1_a1_right_finger_dist_link: geometry collision mesh filename=file:///srv/data/users/raditya/arm_WS/ceiling_arm/ros2_ws/i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; visual mesh filename=file:///srv/data/users/raditya/arm_WS/ceiling_arm/ros2_ws/i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
- link t1_a1_right_finger_prox_link: geometry collision mesh filename=file:///srv/data/users/raditya/arm_WS/ceiling_arm/ros2_ws/i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; visual mesh filename=file:///srv/data/users/raditya/arm_WS/ceiling_arm/ros2_ws/i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
- link t1_a2_gripper_base_link: geometry collision mesh filename=file:///srv/data/users/raditya/arm_WS/ceiling_arm/ros2_ws/i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; visual mesh filename=file:///srv/data/users/raditya/arm_WS/ceiling_arm/ros2_ws/i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
- link t1_a2_left_finger_dist_link: geometry collision mesh filename=file:///srv/data/users/raditya/arm_WS/ceiling_arm/ros2_ws/i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; visual mesh filename=file:///srv/data/users/raditya/arm_WS/ceiling_arm/ros2_ws/i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
- link t1_a2_left_finger_prox_link: geometry collision mesh filename=file:///srv/data/users/raditya/arm_WS/ceiling_arm/ros2_ws/i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; visual mesh filename=file:///srv/data/users/raditya/arm_WS/ceiling_arm/ros2_ws/i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
- link t1_a2_right_finger_dist_link: geometry collision mesh filename=file:///srv/data/users/raditya/arm_WS/ceiling_arm/ros2_ws/i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; visual mesh filename=file:///srv/data/users/raditya/arm_WS/ceiling_arm/ros2_ws/i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
- link t1_a2_right_finger_prox_link: geometry collision mesh filename=file:///srv/data/users/raditya/arm_WS/ceiling_arm/ros2_ws/i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; visual mesh filename=file:///srv/data/users/raditya/arm_WS/ceiling_arm/ros2_ws/i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
- link t2_a1_gripper_base_link: geometry collision mesh filename=file:///srv/data/users/raditya/arm_WS/ceiling_arm/ros2_ws/i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; visual mesh filename=file:///srv/data/users/raditya/arm_WS/ceiling_arm/ros2_ws/i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
- link t2_a1_left_finger_dist_link: geometry collision mesh filename=file:///srv/data/users/raditya/arm_WS/ceiling_arm/ros2_ws/i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; visual mesh filename=file:///srv/data/users/raditya/arm_WS/ceiling_arm/ros2_ws/i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
- link t2_a1_left_finger_prox_link: geometry collision mesh filename=file:///srv/data/users/raditya/arm_WS/ceiling_arm/ros2_ws/i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; visual mesh filename=file:///srv/data/users/raditya/arm_WS/ceiling_arm/ros2_ws/i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
- link t2_a1_right_finger_dist_link: geometry collision mesh filename=file:///srv/data/users/raditya/arm_WS/ceiling_arm/ros2_ws/i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; visual mesh filename=file:///srv/data/users/raditya/arm_WS/ceiling_arm/ros2_ws/i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
- link t2_a1_right_finger_prox_link: geometry collision mesh filename=file:///srv/data/users/raditya/arm_WS/ceiling_arm/ros2_ws/i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; visual mesh filename=file:///srv/data/users/raditya/arm_WS/ceiling_arm/ros2_ws/i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
- link t2_a2_gripper_base_link: geometry collision mesh filename=file:///srv/data/users/raditya/arm_WS/ceiling_arm/ros2_ws/i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; visual mesh filename=file:///srv/data/users/raditya/arm_WS/ceiling_arm/ros2_ws/i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
- link t2_a2_left_finger_dist_link: geometry collision mesh filename=file:///srv/data/users/raditya/arm_WS/ceiling_arm/ros2_ws/i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; visual mesh filename=file:///srv/data/users/raditya/arm_WS/ceiling_arm/ros2_ws/i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
- link t2_a2_left_finger_prox_link: geometry collision mesh filename=file:///srv/data/users/raditya/arm_WS/ceiling_arm/ros2_ws/i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; visual mesh filename=file:///srv/data/users/raditya/arm_WS/ceiling_arm/ros2_ws/i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
- link t2_a2_right_finger_dist_link: geometry collision mesh filename=file:///srv/data/users/raditya/arm_WS/ceiling_arm/ros2_ws/i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; visual mesh filename=file:///srv/data/users/raditya/arm_WS/ceiling_arm/ros2_ws/i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
- link t2_a2_right_finger_prox_link: geometry collision mesh filename=file:///srv/data/users/raditya/arm_WS/ceiling_arm/ros2_ws/i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; visual mesh filename=file:///srv/data/users/raditya/arm_WS/ceiling_arm/ros2_ws/i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
Joints:
- joint t1_a1_base_joint: origin xyz=0 0 -0.025 rpy=3.14159 0 3.14159 -> xyz=0 0 -0.025 rpy=3.14159 0 -1.5707963267948966; parent t1_mount_plate_left -> t1_mount_plate_right
- joint t1_a1_left_finger_bottom_joint: limit lower=-0.96 upper=0.09 effort=10 velocity=0.6 -> lower=-0.1 upper=0.96 effort=10 velocity=0.6; mimic (none) -> joint=t1_a1_right_finger_bottom_joint multiplier=1.0 offset=0.0; origin xyz=0 0.0305 0.070003 rpy=0 1.5708 0 -> xyz=0 0.0305 0.070003 rpy=-1.571 0.611 -1.571
- joint t1_a1_left_finger_tip_joint: mimic (none) -> joint=t1_a1_right_finger_bottom_joint multiplier=-0.276 offset=-0.1
- joint t1_a1_right_finger_bottom_joint: axis 0 0 1 -> 0 0 -1; limit lower=-0.09 upper=0.96 effort=10 velocity=0.6 -> lower=-0.1 upper=0.96 effort=10 velocity=0.6; origin xyz=0 -0.030501 0.070003 rpy=0 1.5708 0 -> xyz=0 -0.030501 0.070003 rpy=1.571 0.611 1.571
- joint t1_a1_right_finger_tip_joint: mimic (none) -> joint=t1_a1_right_finger_bottom_joint multiplier=-0.276 offset=-0.1
- joint t1_a2_base_joint: origin xyz=0 0 -0.025 rpy=3.14159 0 0 -> xyz=0 0 -0.025 rpy=3.14159 0 1.5707963267948966; parent t1_mount_plate_right -> t1_mount_plate_left
- joint t1_a2_left_finger_bottom_joint: limit lower=-0.96 upper=0.09 effort=10 velocity=0.6 -> lower=-0.1 upper=0.96 effort=10 velocity=0.6; mimic (none) -> joint=t1_a2_right_finger_bottom_joint multiplier=1.0 offset=0.0; origin xyz=0 0.0305 0.070003 rpy=0 1.5708 0 -> xyz=0 0.0305 0.070003 rpy=-1.571 0.611 -1.571
- joint t1_a2_left_finger_tip_joint: mimic (none) -> joint=t1_a2_right_finger_bottom_joint multiplier=-0.276 offset=-0.1
- joint t1_a2_right_finger_bottom_joint: axis 0 0 1 -> 0 0 -1; limit lower=-0.09 upper=0.96 effort=10 velocity=0.6 -> lower=-0.1 upper=0.96 effort=10 velocity=0.6; origin xyz=0 -0.030501 0.070003 rpy=0 1.5708 0 -> xyz=0 -0.030501 0.070003 rpy=1.571 0.611 1.571
- joint t1_a2_right_finger_tip_joint: mimic (none) -> joint=t1_a2_right_finger_bottom_joint multiplier=-0.276 offset=-0.1
- joint t1_rotation_joint: limit lower=-3.14159265359 upper=3.14159265359 effort=10 velocity=1.0 -> lower=-3.141592653589793 upper=3.141592653589793 effort=10 velocity=1.0
- joint t2_a1_base_joint: origin xyz=0 0 -0.025 rpy=3.14159 0 3.14159 -> xyz=0 0 -0.025 rpy=3.14159 0 -1.5707963267948966; parent t2_mount_plate_left -> t2_mount_plate_right
- joint t2_a1_left_finger_bottom_joint: limit lower=-0.96 upper=0.09 effort=10 velocity=0.6 -> lower=-0.1 upper=0.96 effort=10 velocity=0.6; mimic (none) -> joint=t2_a1_right_finger_bottom_joint multiplier=1.0 offset=0.0; origin xyz=0 0.0305 0.070003 rpy=0 1.5708 0 -> xyz=0 0.0305 0.070003 rpy=-1.571 0.611 -1.571
- joint t2_a1_left_finger_tip_joint: mimic (none) -> joint=t2_a1_right_finger_bottom_joint multiplier=-0.276 offset=-0.1
- joint t2_a1_right_finger_bottom_joint: axis 0 0 1 -> 0 0 -1; limit lower=-0.09 upper=0.96 effort=10 velocity=0.6 -> lower=-0.1 upper=0.96 effort=10 velocity=0.6; origin xyz=0 -0.030501 0.070003 rpy=0 1.5708 0 -> xyz=0 -0.030501 0.070003 rpy=1.571 0.611 1.571
- joint t2_a1_right_finger_tip_joint: mimic (none) -> joint=t2_a1_right_finger_bottom_joint multiplier=-0.276 offset=-0.1
- joint t2_a2_base_joint: origin xyz=0 0 -0.025 rpy=3.14159 0 0 -> xyz=0 0 -0.025 rpy=3.14159 0 1.5707963267948966; parent t2_mount_plate_right -> t2_mount_plate_left
- joint t2_a2_left_finger_bottom_joint: limit lower=-0.96 upper=0.09 effort=10 velocity=0.6 -> lower=-0.1 upper=0.96 effort=10 velocity=0.6; mimic (none) -> joint=t2_a2_right_finger_bottom_joint multiplier=1.0 offset=0.0; origin xyz=0 0.0305 0.070003 rpy=0 1.5708 0 -> xyz=0 0.0305 0.070003 rpy=-1.571 0.611 -1.571
- joint t2_a2_left_finger_tip_joint: mimic (none) -> joint=t2_a2_right_finger_bottom_joint multiplier=-0.276 offset=-0.1
- joint t2_a2_right_finger_bottom_joint: axis 0 0 1 -> 0 0 -1; limit lower=-0.09 upper=0.96 effort=10 velocity=0.6 -> lower=-0.1 upper=0.96 effort=10 velocity=0.6; origin xyz=0 -0.030501 0.070003 rpy=0 1.5708 0 -> xyz=0 -0.030501 0.070003 rpy=1.571 0.611 1.571
- joint t2_a2_right_finger_tip_joint: mimic (none) -> joint=t2_a2_right_finger_bottom_joint multiplier=-0.276 offset=-0.1
- joint t2_rotation_joint: limit lower=-1.57 upper=1.57 effort=10 velocity=1.0 -> lower=-3.141592653589793 upper=3.141592653589793 effort=10 velocity=1.0

Commit message: fix(safety): rail travel limit is 1600mm, not 2000 -- and the service path had no guard
The gantry ran into the rail end stop on 2026-08-13 while a move to 1900mm was
executing (docs/p1_g3_timing.md B3b). The end stop is at ~1656mm from encoder
zero; 1600mm is the operational limit (56mm margin).

Three places promised travel that does not physically exist:
  - bridge.max_mm            2000.0 -> 1600.0
  - moving_table.urdf.xacro  upper 2.0 -> 1.6
  - workcell_full.urdf       upper 2.0 -> 1.6  (x2, used by the offline tools)

And a fourth, which is how the crash actually got dispatched: the
move_dual_table SERVICE path had no range check at all. Only the ros2_control
bridge validated against bridge.min_mm/max_mm. Added _check_travel_limits(),
which resolves the request to an ABSOLUTE target first -- go_to_table is a
RELATIVE move (moving_table.py:100 adds the increment to the live encoder
reading), so a small-looking delta can still land past the end stop.

Verified 11 cases offline, including the exact crash command (ABS 1900 ->
REJECT) and the relative case (+1100mm from 550 -> 1650 -> REJECT) that the
old code dispatched without complaint. Then verified on live hardware with
max_mm temporarily lowered to 600 so a guard failure would have been harmless:
rejected before the move thread was created, zero Modbus writes, encoder
bit-identical at 52519 pulses.

Jog (op 10-13) is still NOT range-checked: it is continuous and has no target,
so it cannot be. Left open deliberately -- it is the human-in-the-loop tool and
is not on the scheduler's path -- but it now warns within 100mm of the limits.

irm_sweep: RAIL_MAX_M = 1.60 is now the make_grid default, so capability sweeps
stop generating gantry poses that cannot be reached. Maps swept before today
used 0..2.0m, i.e. 8 of 41 linear columns are phantom.

Co-Authored-By: Claude Opus 5 <noreply@anthropic.com>

File: ros2_ws/src/workcell_description/urdf/moving_table.urdf.xacro (robot description, xacro)
@@ -31,5 +31,9 @@
       </inertial>
     </link>
-    <!-- Linear slide -->
+    <!-- Linear slide.
+         upper=1.6, NOT 2.0: the rail end stop was MEASURED at ~1.656 m from
+         encoder zero on 2026-08-13 (the gantry hit it; docs/p1_g3_timing.md
+         §B3b). The old 2.0 promised ~0.34 m of travel that does not physically
+         exist, so MoveIt would happily plan gantry poses into the end stop. -->
     <joint name="${prefix}linear_joint" type="prismatic">
       <parent link="${prefix}base_link"/>
@@ -37,5 +41,5 @@
       <origin xyz="0 0 0" rpy="0 0 0"/>
       <axis xyz="1 0 0"/>
-      <limit lower="0.0" upper="2.0" effort="1000" velocity="0.5"/>
+      <limit lower="0.0" upper="1.6" effort="1000" velocity="0.5"/>
     </joint>
     <!-- Rotation bar -->

File: ros2_ws/src/workcell_description/urdf/workcell_full.urdf (robot description, URDF)
Before this commit: robot trailer_workcell, 67 links, 66 joints
Joints:
- joint t1_linear_joint: limit lower=0.0 upper=2.0 effort=1000 velocity=0.5 -> lower=0.0 upper=1.6 effort=1000 velocity=0.5
- joint t2_linear_joint: limit lower=0.0 upper=2.0 effort=1000 velocity=0.5 -> lower=0.0 upper=1.6 effort=1000 velocity=0.5
