Commit message: Enhance kinematics configuration and trajectory execution settings
- Added kinematics solver configurations for gantry_2_with_arm_1 and gantry_2_with_arm_2 in kinematics.yaml.
- Increased trajectory execution duration scaling and goal duration margin in my_workcell.launch.py to accommodate slower execution in Isaac physics.
- Introduced a new TypeScript file mobileclip_blt.ts, which is currently too large to diff.

File: ros2_ws/src/workcell_description/urdf/workcell_full.urdf (robot description, URDF)
Before this commit: robot trailer_workcell, 67 links, 66 joints
Links:
- link t1_a1_arm_link: geometry collision mesh filename=file:///srv/data/users/raditya/kortex_min_ws/install/kortex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; visual mesh filename=file:///srv/data/users/raditya/kortex_min_ws/install/kortex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
- link t1_a1_base_link: geometry collision mesh filename=file:///srv/data/users/raditya/kortex_min_ws/install/kortex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; visual mesh filename=file:///srv/data/users/raditya/kortex_min_ws/install/kortex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
- link t1_a1_forearm_link: geometry collision mesh filename=file:///srv/data/users/raditya/kortex_min_ws/install/kortex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; visual mesh filename=file:///srv/data/users/raditya/kortex_min_ws/install/kortex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
- link t1_a1_gripper_base_link: geometry collision mesh filename=file:///srv/data/users/raditya/kortex_min_ws/install/kortex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; visual mesh filename=file:///srv/data/users/raditya/kortex_min_ws/install/kortex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
- link t1_a1_left_finger_dist_link: geometry collision mesh filename=file:///srv/data/users/raditya/kortex_min_ws/install/kortex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; visual mesh filename=file:///srv/data/users/raditya/kortex_min_ws/install/kortex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
- link t1_a1_left_finger_prox_link: geometry collision mesh filename=file:///srv/data/users/raditya/kortex_min_ws/install/kortex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; visual mesh filename=file:///srv/data/users/raditya/kortex_min_ws/install/kortex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
- link t1_a1_lower_wrist_link: geometry collision mesh filename=file:///srv/data/users/raditya/kortex_min_ws/install/kortex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; visual mesh filename=file:///srv/data/users/raditya/kortex_min_ws/install/kortex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
- link t1_a1_right_finger_dist_link: geometry collision mesh filename=file:///srv/data/users/raditya/kortex_min_ws/install/kortex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; visual mesh filename=file:///srv/data/users/raditya/kortex_min_ws/install/kortex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
- link t1_a1_right_finger_prox_link: geometry collision mesh filename=file:///srv/data/users/raditya/kortex_min_ws/install/kortex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; visual mesh filename=file:///srv/data/users/raditya/kortex_min_ws/install/kortex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
- link t1_a1_shoulder_link: geometry collision mesh filename=file:///srv/data/users/raditya/kortex_min_ws/install/kortex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; visual mesh filename=file:///srv/data/users/raditya/kortex_min_ws/install/kortex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
- link t1_a1_upper_wrist_link: geometry collision mesh filename=file:///srv/data/users/raditya/kortex_min_ws/install/kortex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; visual mesh filename=file:///srv/data/users/raditya/kortex_min_ws/install/kortex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
- link t1_a2_arm_link: geometry collision mesh filename=file:///srv/data/users/raditya/kortex_min_ws/install/kortex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; visual mesh filename=file:///srv/data/users/raditya/kortex_min_ws/install/kortex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
- link t1_a2_base_link: geometry collision mesh filename=file:///srv/data/users/raditya/kortex_min_ws/install/kortex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; visual mesh filename=file:///srv/data/users/raditya/kortex_min_ws/install/kortex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
- link t1_a2_forearm_link: geometry collision mesh filename=file:///srv/data/users/raditya/kortex_min_ws/install/kortex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; visual mesh filename=file:///srv/data/users/raditya/kortex_min_ws/install/kortex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
- link t1_a2_gripper_base_link: geometry collision mesh filename=file:///srv/data/users/raditya/kortex_min_ws/install/kortex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; visual mesh filename=file:///srv/data/users/raditya/kortex_min_ws/install/kortex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
- link t1_a2_left_finger_dist_link: geometry collision mesh filename=file:///srv/data/users/raditya/kortex_min_ws/install/kortex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; visual mesh filename=file:///srv/data/users/raditya/kortex_min_ws/install/kortex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
- link t1_a2_left_finger_prox_link: geometry collision mesh filename=file:///srv/data/users/raditya/kortex_min_ws/install/kortex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; visual mesh filename=file:///srv/data/users/raditya/kortex_min_ws/install/kortex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
- link t1_a2_lower_wrist_link: geometry collision mesh filename=file:///srv/data/users/raditya/kortex_min_ws/install/kortex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; visual mesh filename=file:///srv/data/users/raditya/kortex_min_ws/install/kortex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
- link t1_a2_right_finger_dist_link: geometry collision mesh filename=file:///srv/data/users/raditya/kortex_min_ws/install/kortex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; visual mesh filename=file:///srv/data/users/raditya/kortex_min_ws/install/kortex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
- link t1_a2_right_finger_prox_link: geometry collision mesh filename=file:///srv/data/users/raditya/kortex_min_ws/install/kortex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; visual mesh filename=file:///srv/data/users/raditya/kortex_min_ws/install/kortex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
- link t1_a2_shoulder_link: geometry collision mesh filename=file:///srv/data/users/raditya/kortex_min_ws/install/kortex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; visual mesh filename=file:///srv/data/users/raditya/kortex_min_ws/install/kortex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
- link t1_a2_upper_wrist_link: geometry collision mesh filename=file:///srv/data/users/raditya/kortex_min_ws/install/kortex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; visual mesh filename=file:///srv/data/users/raditya/kortex_min_ws/install/kortex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
- link t2_a1_arm_link: geometry collision mesh filename=file:///srv/data/users/raditya/kortex_min_ws/install/kortex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; visual mesh filename=file:///srv/data/users/raditya/kortex_min_ws/install/kortex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
- link t2_a1_base_link: geometry collision mesh filename=file:///srv/data/users/raditya/kortex_min_ws/install/kortex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; visual mesh filename=file:///srv/data/users/raditya/kortex_min_ws/install/kortex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
- link t2_a1_forearm_link: geometry collision mesh filename=file:///srv/data/users/raditya/kortex_min_ws/install/kortex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; visual mesh filename=file:///srv/data/users/raditya/kortex_min_ws/install/kortex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
- link t2_a1_gripper_base_link: geometry collision mesh filename=file:///srv/data/users/raditya/kortex_min_ws/install/kortex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; visual mesh filename=file:///srv/data/users/raditya/kortex_min_ws/install/kortex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
- link t2_a1_left_finger_dist_link: geometry collision mesh filename=file:///srv/data/users/raditya/kortex_min_ws/install/kortex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; visual mesh filename=file:///srv/data/users/raditya/kortex_min_ws/install/kortex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
- link t2_a1_left_finger_prox_link: geometry collision mesh filename=file:///srv/data/users/raditya/kortex_min_ws/install/kortex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; visual mesh filename=file:///srv/data/users/raditya/kortex_min_ws/install/kortex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
- link t2_a1_lower_wrist_link: geometry collision mesh filename=file:///srv/data/users/raditya/kortex_min_ws/install/kortex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; visual mesh filename=file:///srv/data/users/raditya/kortex_min_ws/install/kortex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
- link t2_a1_right_finger_dist_link: geometry collision mesh filename=file:///srv/data/users/raditya/kortex_min_ws/install/kortex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; visual mesh filename=file:///srv/data/users/raditya/kortex_min_ws/install/kortex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
- link t2_a1_right_finger_prox_link: geometry collision mesh filename=file:///srv/data/users/raditya/kortex_min_ws/install/kortex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; visual mesh filename=file:///srv/data/users/raditya/kortex_min_ws/install/kortex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
- link t2_a1_shoulder_link: geometry collision mesh filename=file:///srv/data/users/raditya/kortex_min_ws/install/kortex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; visual mesh filename=file:///srv/data/users/raditya/kortex_min_ws/install/kortex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
- link t2_a1_upper_wrist_link: geometry collision mesh filename=file:///srv/data/users/raditya/kortex_min_ws/install/kortex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; visual mesh filename=file:///srv/data/users/raditya/kortex_min_ws/install/kortex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
- link t2_a2_arm_link: geometry collision mesh filename=file:///srv/data/users/raditya/kortex_min_ws/install/kortex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; visual mesh filename=file:///srv/data/users/raditya/kortex_min_ws/install/kortex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
- link t2_a2_base_link: geometry collision mesh filename=file:///srv/data/users/raditya/kortex_min_ws/install/kortex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; visual mesh filename=file:///srv/data/users/raditya/kortex_min_ws/install/kortex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
- link t2_a2_forearm_link: geometry collision mesh filename=file:///srv/data/users/raditya/kortex_min_ws/install/kortex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; visual mesh filename=file:///srv/data/users/raditya/kortex_min_ws/install/kortex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
- link t2_a2_gripper_base_link: geometry collision mesh filename=file:///srv/data/users/raditya/kortex_min_ws/install/kortex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; visual mesh filename=file:///srv/data/users/raditya/kortex_min_ws/install/kortex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
- link t2_a2_left_finger_dist_link: geometry collision mesh filename=file:///srv/data/users/raditya/kortex_min_ws/install/kortex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; visual mesh filename=file:///srv/data/users/raditya/kortex_min_ws/install/kortex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
- link t2_a2_left_finger_prox_link: geometry collision mesh filename=file:///srv/data/users/raditya/kortex_min_ws/install/kortex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; visual mesh filename=file:///srv/data/users/raditya/kortex_min_ws/install/kortex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
- link t2_a2_lower_wrist_link: geometry collision mesh filename=file:///srv/data/users/raditya/kortex_min_ws/install/kortex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; visual mesh filename=file:///srv/data/users/raditya/kortex_min_ws/install/kortex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
- link t2_a2_right_finger_dist_link: geometry collision mesh filename=file:///srv/data/users/raditya/kortex_min_ws/install/kortex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; visual mesh filename=file:///srv/data/users/raditya/kortex_min_ws/install/kortex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
- link t2_a2_right_finger_prox_link: geometry collision mesh filename=file:///srv/data/users/raditya/kortex_min_ws/install/kortex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; visual mesh filename=file:///srv/data/users/raditya/kortex_min_ws/install/kortex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
- link t2_a2_shoulder_link: geometry collision mesh filename=file:///srv/data/users/raditya/kortex_min_ws/install/kortex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; visual mesh filename=file:///srv/data/users/raditya/kortex_min_ws/install/kortex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
- link t2_a2_upper_wrist_link: geometry collision mesh filename=file:///srv/data/users/raditya/kortex_min_ws/install/kortex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; visual mesh filename=file:///srv/data/users/raditya/kortex_min_ws/install/kortex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
Joints:
- joint t1_a1_base_joint: origin xyz=0 0 -0.025 rpy=3.14159 0 3.14159 -> xyz=0 0 -0.025 rpy=3.14159 0 -1.5707963267948966; parent t1_mount_plate_left -> t1_mount_plate_right
- joint t1_a2_base_joint: origin xyz=0 0 -0.025 rpy=3.14159 0 0 -> xyz=0 0 -0.025 rpy=3.14159 0 1.5707963267948966; parent t1_mount_plate_right -> t1_mount_plate_left
- joint t1_rotation_joint: limit lower=-3.14159265359 upper=3.14159265359 effort=10 velocity=1.0 -> lower=-3.141592653589793 upper=3.141592653589793 effort=10 velocity=1.0
- joint t2_a1_base_joint: origin xyz=0 0 -0.025 rpy=3.14159 0 3.14159 -> xyz=0 0 -0.025 rpy=3.14159 0 -1.5707963267948966; parent t2_mount_plate_left -> t2_mount_plate_right
- joint t2_a2_base_joint: origin xyz=0 0 -0.025 rpy=3.14159 0 0 -> xyz=0 0 -0.025 rpy=3.14159 0 1.5707963267948966; parent t2_mount_plate_right -> t2_mount_plate_left
- joint t2_rotation_joint: limit lower=-1.57 upper=1.57 effort=10 velocity=1.0 -> lower=-3.141592653589793 upper=3.141592653589793 effort=10 velocity=1.0
