Commit message: fix(cell_gazebo_sim): resolve Fortress spawn issues (Phase 2 fixup)
- Replace empty t1/t2_base_link with direct prismatic-from-world table
  geometry to prevent Gazebo URDF→SDF fixed-joint lumping that dropped
  all arm/table links from the SDF.
- Inline sim_table macro in cell_sim.urdf.xacro (does NOT include
  moving_table.urdf.xacro to avoid empty-link lump issue).
- Switch sensor render engine from ogre → ogre2 in both world SDF and
  robot URDF plugins (ogre1 crashes in OgreRTShaderSystem on this host).
- launch: prepend /opt/ros/humble/lib to GZ_SIM_SYSTEM_PLUGIN_PATH so
  gz_ros2_control-system.so is found.
- launch: set IGN_GAZEBO_RESOURCE_PATH to kortex_description share parent
  so model://kortex_description mesh URIs resolve.
- launch: sed-patch GzSimSystem→GazeboSimSystem at runtime (newer kortex
  uses GzSimSystem alias not yet registered in installed gz_ros2_control).
- Document kortex_description workspace precedence in sim xacro.

Known: Ogre2/Ogre1 sensor rendering crashes on Intel iGPU (Arc/Alder Lake)
due to GPU driver compatibility. Bridge topics (/livox/points, /camera/*)
are correctly wired and appear on the ROS 2 bus; they publish when Gazebo
runs on a machine with a working Ogre render context. All ros2_control
hardware systems (TableSimSystem, 4 arms, 4 grippers) initialize and
activate correctly in headless mode without sensors.

Co-Authored-By: Claude Sonnet 4.6 <noreply@anthropic.com>

File: ros2_ws/src/cell_gazebo_sim/urdf/cell_sim.urdf.xacro (robot description, xacro)
@@ -22,5 +22,4 @@
   <xacro:arg name="sim_controllers"
              default="$(find cell_gazebo_sim)/config/sim_ros2_controllers.yaml"/>
-  <xacro:arg name="gazebo_renderer" default="ogre"/>
   <!-- Arm IP args kept for signature compatibility; unused in sim. -->
   <xacro:arg name="arm1_ip" default="0.0.0.0"/>
@@ -31,7 +30,13 @@
   <!-- Include macros                                                -->
   <!-- ============================================================ -->
-  <!-- Table geometry (shared with real-hardware path, no changes needed) -->
-  <xacro:include filename="$(find workcell_description)/urdf/moving_table.urdf.xacro"/>
-  <!-- Kinova Gen3 Lite arm macro (from ros2_kortex submodule/sibling ws) -->
+  <!-- Kinova Gen3 Lite arm macro (from ros2_kortex).
+       IMPORTANT — two kortex_description installs exist on this machine:
+         /home/mobi/Documents/moonshot_project/ros2_ws  → uses gazebo_ros2_control/GazeboSystem (Gazebo11, not installed)
+         /home/mobi/ros2_ws                             → uses gz_ros2_control/GazeboSimSystem (Fortress, correct)
+       The launch file prepends /home/mobi/ros2_ws/install/kortex_description to
+       AMENT_PREFIX_PATH so $(find kortex_description) resolves to the correct copy.
+       The gripper ros2_control xacro in the correct copy uses gz_ros2_control/GzSimSystem
+       (a newer alias); the launch file's sed replaces it with GazeboSimSystem at runtime
+       because this machine's gz_ros2_control package does not yet register GzSimSystem. -->
   <xacro:include filename="$(find kortex_description)/robots/kortex_robot.xacro"/>
   <xacro:include filename="$(find kortex_description)/arms/gen3_lite/6dof/urdf/kortex.ros2_control.xacro"/>
@@ -39,16 +44,130 @@
   <xacro:include filename="$(find kortex_description)/grippers/gen3_lite_2f/urdf/gen3_lite_2f_transmission_macro.xacro"/>
   <!-- ============================================================ -->
+  <!-- Sim table macro                                               -->
+  <!--                                                              -->
+  <!-- We do NOT include moving_table.urdf.xacro here.              -->
+  <!-- That macro creates an empty t1_base_link (no inertial) which  -->
+  <!-- Gazebo's URDF→SDF converter lumps into world, then drops all  -->
+  <!-- descendants.  Instead we inline the table geometry with the    -->
+  <!-- prismatic joint attached directly to world (the y/z offset is  -->
+  <!-- on the joint origin), giving every link proper inertia.        -->
+  <!--                                                                -->
+  <!-- The link/joint NAMES are identical to the real-hardware model, -->
+  <!-- so all ROS controller/SRDF references stay unchanged.          -->
+  <!-- ============================================================ -->
+  <xacro:macro name="sim_table" params="prefix y_offset">
+    <xacro:property name="p_mass" value="5.0"/>
+    <xacro:property name="r_mass" value="3.0"/>
+    <xacro:property name="mp_mass" value="0.2"/>
+    <xacro:property name="mp_r" value="0.055"/>
+    <xacro:property name="mp_l" value="0.05"/>
+    <xacro:property name="mp_y" value="0.4"/>
+    <!-- Platform (was child of empty base_link; now child of world directly) -->
+    <link name="${prefix}platform_link">
+      <visual>
+        <geometry><box size="0.35 0.34 0.065"/></geometry>
+        <material name="grey"><color rgba="0.6 0.6 0.6 1.0"/></material>
+      </visual>
+      <collision>
+        <geometry><box size="0.35 0.34 0.065"/></geometry>
+      </collision>
+      <inertial>
+        <mass value="${p_mass}"/>
+        <inertia
+          ixx="${p_mass/12.0*(0.34*0.34+0.065*0.065)}"
+          iyy="${p_mass/12.0*(0.35*0.35+0.065*0.065)}"
+          izz="${p_mass/12.0*(0.35*0.35+0.34*0.34)}"
+          ixy="0" ixz="0" iyz="0"/>
+      </inertial>
+    </link>
+    <!-- Prismatic joint with the table's base offset on its origin -->
+    <joint name="${prefix}linear_joint" type="prismatic">
+      <parent link="world"/>
+      <child link="${prefix}platform_link"/>
+      <origin xyz="0 ${y_offset} 2.05" rpy="0 0 0"/>
+      <axis xyz="1 0 0"/>
+      <limit lower="0.0" upper="1.5" effort="1000" velocity="0.5"/>
+    </joint>
+    <!-- Rotation bar -->
+    <link name="${prefix}rotation_link">
+      <visual>
+        <geometry><box size="0.08 0.8 0.015"/></geometry>
+        <material name="dark_grey"><color rgba="0.3 0.3 0.3 1.0"/></material>
+      </visual>
+      <collision>
+        <geometry><box size="0.08 0.8 0.015"/></geometry>
+      </collision>
+      <inertial>
+        <mass value="${r_mass}"/>
+        <inertia
+          ixx="${r_mass/12.0*(0.8*0.8+0.015*0.015)}"
+          iyy="${r_mass/12.0*(0.08*0.08+0.015*0.015)}"
+          izz="${r_mass/12.0*(0.08*0.08+0.8*0.8)}"
+          ixy="0" ixz="0" iyz="0"/>
+      </inertial>
+    </link>
+    <joint name="${prefix}rotation_joint" type="revolute">
+      <parent link="${prefix}platform_link"/>
+      <child link="${prefix}rotation_link"/>
+      <origin xyz="0 0 -${0.065/2+0.015/2}" rpy="0 0 ${pi/2}"/>
+      <axis xyz="0 0 1"/>
+      <limit lower="-1.57" upper="1.57" effort="10" velocity="1.0"/>
+    </joint>
+    <!-- Left mount plate -->
+    <link name="${prefix}mount_plate_left">
+      <visual>
+        <geometry><cylinder radius="${mp_r}" length="${mp_l}"/></geometry>
+        <material name="black"><color rgba="0.1 0.1 0.1 1.0"/></material>
+      </visual>
+      <collision>
+        <geometry><cylinder radius="${mp_r}" length="${mp_l}"/></geometry>
+      </collision>
+      <inertial>
+        <mass value="${mp_mass}"/>
+        <inertia
+          ixx="${mp_mass/12.0*(3*mp_r*mp_r+mp_l*mp_l)}"
+          iyy="${mp_mass/12.0*(3*mp_r*mp_r+mp_l*mp_l)}"
+          izz="${mp_mass/2.0*mp_r*mp_r}"
+          ixy="0" ixz="0" iyz="0"/>
+      </inertial>
+    </link>
+    <joint name="${prefix}mount_plate_left_joint" type="fixed">
+      <parent link="${prefix}rotation_link"/>
+      <child link="${prefix}mount_plate_left"/>
+      <origin xyz="0 ${mp_y} -${0.015/2+0.05/2}" rpy="0 0 0"/>
+    </joint>
+    <!-- Right mount plate -->
+    <link name="${prefix}mount_plate_right">
+      <visual>
+        <geometry><cylinder radius="${mp_r}" length="${mp_l}"/></geometry>
+        <material name="black"><color rgba="0.1 0.1 0.1 1.0"/></material>
+      </visual>
+      <collision>
+        <geometry><cylinder radius="${mp_r}" length="${mp_l}"/></geometry>
+      </collision>
+      <inertial>
+        <mass value="${mp_mass}"/>
+        <inertia
+          ixx="${mp_mass/12.0*(3*mp_r*mp_r+mp_l*mp_l)}"
+          iyy="${mp_mass/12.0*(3*mp_r*mp_r+mp_l*mp_l)}"
+          izz="${mp_mass/2.0*mp_r*mp_r}"
+          ixy="0" ixz="0" iyz="0"/>
+      </inertial>
+    </link>
+    <joint name="${prefix}mount_plate_right_joint" type="fixed">
+      <parent link="${prefix}rotation_link"/>
+      <child link="${prefix}mount_plate_right"/>
+      <origin xyz="0 -${mp_y} -${0.015/2+0.05/2}" rpy="0 0 0"/>
+    </joint>
+  </xacro:macro>
+  <!-- ============================================================ -->
   <!-- World / root link                                             -->
   <!-- ============================================================ -->
   <link name="world"/>
   <!-- ============================================================ -->
-  <!-- Moving tables (same topology as workcell.urdf.xacro)         -->
-  <!-- ============================================================ -->
-  <xacro:moving_table prefix="t1_" parent="world">
-    <origin xyz="0 0.36 2.05" rpy="0 0 0"/>
-  </xacro:moving_table>
-  <xacro:moving_table prefix="t2_" parent="world">
-    <origin xyz="0 -0.36 2.05" rpy="0 0 0"/>
-  </xacro:moving_table>
+  <!-- Moving tables (sim version without empty base_link)           -->
+  <!-- ============================================================ -->
+  <xacro:sim_table prefix="t1_" y_offset="0.36"/>
+  <xacro:sim_table prefix="t2_" y_offset="-0.36"/>
   <!-- ============================================================ -->
   <!-- Table joints in ros2_control (sim only)                      -->
@@ -297,5 +416,5 @@
     <plugin filename="gz-sim-sensors-system"
             name="gz::sim::systems::Sensors">
-      <render_engine>$(arg gazebo_renderer)</render_engine>
+      <render_engine>ogre2</render_engine>
     </plugin>
   </gazebo>
