Commit message: Add reachability_gng package with GNG map generation and visualization
- Create README.html for package documentation, detailing setup and usage instructions.
- Implement build_maps.sh script for generating GNG reachability maps for multiple arms.
- Add configuration file for arm2_table1.yaml to define sampling parameters for the second arm.
- Create gng_moveit.rviz configuration for visualizing GNG clouds alongside MoveIt planning.
- Develop launch files gng_clouds.launch.py and gng_moveit.launch.py to facilitate running the GNG visualization and MoveIt planning in a single RViz instance.

File: isaac_sim/workcell/workcell.urdf (robot description, URDF)
Before this commit: robot trailer_workcell, 67 links, 66 joints
Joints:
- joint t1_linear_joint: limit lower=0.0 upper=1.5 effort=1000 velocity=0.5 -> lower=0.0 upper=3.0 effort=5000 velocity=0.5
- joint t1_rotation_joint: limit lower=-1.57 upper=1.57 effort=10 velocity=1.0 -> lower=-3.14159 upper=3.14159 effort=500 velocity=1.0
- joint t2_linear_joint: limit lower=0.0 upper=1.5 effort=1000 velocity=0.5 -> lower=0.0 upper=3.0 effort=5000 velocity=0.5
- joint t2_rotation_joint: limit lower=-1.57 upper=1.57 effort=10 velocity=1.0 -> lower=-3.14159 upper=3.14159 effort=500 velocity=1.0

File: ros2_ws/src/workcell_description/urdf/moving_table.urdf.xacro (robot description, xacro)
@@ -68,5 +68,5 @@
       <origin xyz="0 0 -${0.065/2 + 0.015/2}" rpy="0 0 ${pi/2}"/> <!-- default 90° -->
       <axis xyz="0 0 1"/> <!-- rotate around Z -->
-      <limit lower="-1.57" upper="1.57" effort="10" velocity="1.0"/> <!-- example ±90° -->
+      <limit lower="${-pi}" upper="${pi}" effort="10" velocity="1.0"/> <!-- ±180° travel -->
     </joint>
     <!-- ========== Mount plates (Arm attachment points) ========== -->

File: ros2_ws/src/workcell_description/urdf/workcell.urdf.xacro (robot description, xacro)
@@ -87,5 +87,9 @@
       <hardware>
         <plugin>topic_based_ros2_control/TopicBasedSystem</plugin>
-        <param name="joint_commands_topic">/isaac_joint_commands</param>
+        <!-- Dedicated command topic so the table is NOT starved by the arm/gripper
+             flood on /isaac_joint_commands (the bridge has a separate subscriber
+             for this). States stay on the shared /isaac_joint_states (single
+             publisher = Isaac, no contention). -->
+        <param name="joint_commands_topic">/isaac_table_commands</param>
         <param name="joint_states_topic">/isaac_joint_states</param>
       </hardware>

File: ros2_ws/src/workcell_description/urdf/workcell_full.urdf (robot description, URDF)
Before this commit: robot trailer_workcell, 67 links, 66 joints
Joints:
- joint t1_base_joint: origin xyz=0 0.36 0 rpy=0 0 0 -> xyz=0 0.36 2.05 rpy=0 0 0
- joint t1_rotation_joint: limit lower=-1.57 upper=1.57 effort=10 velocity=1.0 -> lower=-3.14159265359 upper=3.14159265359 effort=10 velocity=1.0
- joint t2_base_joint: origin xyz=0 -0.36 0 rpy=0 0 0 -> xyz=0 -0.36 2.05 rpy=0 0 0
